File: Arduino_MountingHole.pretty/first.kicad_sch (KiCad schematic)
At the start: 22 parts, among them J1 Conn_01x05, J2 Conn_01x04, J3 Conn_01x04, J4 МОТОР А, J5 МОТОР В, J6 UART, J7 BOOT, SW1 SW_SPST, SW2 SW_Push, U1 ESP32-S3-CAM (left), U2 ESP32-S3-CAM (RIGHT), U3 Conn_01x08, U4 Conn_01x08

Commit message: Add firmware: Wi-Fi AP, camera stream, joystick, motors
Connections:
- net IO43 (TX) is gone; now on net ESP_TX: U1.2 (Pin_2)
Other:
- note added: "Камера OV2640 вставляється в роз'єм FPC на платі, її сигнали розведені на самій платі."
- title: (none) -> ринципова схема робота-автомобіля на ESP32-S3-CAM
Changed lines of the file:
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@@
 	(paper "A4")
 	(title_block
+		(title "ринципова схема робота-автомобіля на ESP32-S3-CAM")
 		(date "mar. 31 mars 2015")
 	)
@@
 		)
 	)
+	(text "Камера OV2640 вставляється в роз'єм FPC на платі, її сигнали розведені на самій платі."
+		(exclude_from_sim no)
+		(at 127.254 114.554 0)
+		(effects
+			(font
+				(size 1.27 1.27)
+			)
+		)
+	)
 	(junction
 		(at 152.4 57.15)
@@
 		)
 	)
-	(label "IO43 (TX)"
+	(label "ESP_TX"
 		(at 105.41 95.25 0)
 		(effects
